File: shortKeyboard_sch/shortKeyboard_sch.kicad_pcb (KiCad board)
At the start: 2 copper layers, 41 x 131 mm, 43 parts, among them J1 PH2.0-4, J2 PH2.0-2, J3 PH2.0-2, J4 WF-8, J5 PH2.0-5, J6 PH2.0-2, Q1 SS8050, Q2 SS8050, Q3 AO3401A, U1 CH340G, U3 AMS1117-3.3, U4 ESP32-WROVER, Y1 12M

Commit message: v1.0 commit
Parts:
- moved C4 69.4 mm to (50.1, 149.5), turned to -90 degrees
- moved R17 2.01 mm to (46.8, 77.7)
Routing:
- net GND: track 98.1 -> 87.2 mm
- net +3V3: track 164.6 -> 159.1 mm, vias 2 -> 3
- net /Корневой лист/DTR: track 34.7 -> 36.7 mm
- net /Корневой лист/RTS: track 21.9 -> 23.4 mm
- net Net-(U4-VDD): track 10.2 -> 10.7 mm

Commit message: update pcb(1117->ap2112) + readme images
Parts:
- removed U3: AMS1117-3.3, Package_TO_SOT_SMD:SOT-223-3_TabPin2
- added U5: AP2112K-3.3, Package_TO_SOT_SMD:SOT-23-5, B.Cu at (61.5, 50.6)
Routing:
- net GND: track 87.2 -> 96.3 mm
- net +Vin_AfterSW: track 38.3 -> 43.4 mm
- net +3V3: track 159.1 -> 157.4 mm
